File: coolschematic.kicad_sch (KiCad schematic)
At the start: 38 parts, among them IC1 DRV8825, IC2 DRV8825, J1 1706730, J2 1706730, J3 1706730, J4 1935187, J5 1706730, J6 GP1A57HRJ00F, J7 1935187, J8 GP1A57HRJ00F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

Commit message: Fix naming
Parts:
- D2: value MLBAWT-A1-0000-000W51 -> MLBAWT-A1-0000-000W51
Changed lines of the file:
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@@
       (effects (font (size 1.27 1.27)) (justify right))
     )
-    (property "Value" " MLBAWT-A1-0000-000W51" (id 1) (at 90.17 203.2 90)
+    (property "Value" "MLBAWT-A1-0000-000W51" (id 1) (at 90.17 203.2 90)
       (effects (font (size 1.27 1.27)) (justify right))
     )
@@
     )
     (path "/3bb58e6c-4570-4b7d-8142-aa8f511aa0da"
-      (reference "D2") (unit 1) (value " MLBAWT-A1-0000-000W51") (footprint "LED_SMD:LED_1206_3216Metric_Pad1.42x1.75mm_HandSolder")
+      (reference "D2") (unit 1) (value "MLBAWT-A1-0000-000W51") (footprint "LED_SMD:LED_1206_3216Metric_Pad1.42x1.75mm_HandSolder")
     )
     (path "/216d0c79-c9ad-446e-bf37-485eb452350b"
